Commit message: Replaced file Replaced with URDF obtained from Baxter parameter server

File: files/baxter.urdf (robot description, URDF)
Before this commit: robot baxter, 57 links, 56 joints
Links:
- added link left_gripper_mass, mass 0.000100000000000000
- added link left_gripper_object_mass, mass 0.000100000000000000
- added link right_gripper_mass, mass 0.000100000000000000
- added link right_gripper_object_mass, mass 0.000100000000000000
- link l_gripper_l_finger_tip: geometry collision cylinder length=0.037 radius=0.008; visual mesh filename=package://rethink_ee_description/meshes/electric_gripper/fi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
- link l_gripper_r_finger_tip: geometry collision cylinder length=0.037 radius=0.008; visual mesh filename=package://rethink_ee_description/meshes/electric_gripper/fi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
- link pedestal: geometry collision box size=0.92 0.83 0.3; visual mesh filename=package://baxter_description/meshes/base/PEDESTAL.DAE
- link r_gripper_l_finger: geometry collision box size=0.01 0.0135 0.1127; collision box size=0.01 0.05 0.017
- link r_gripper_l_finger_tip: geometry collision cylinder length=0.037 radius=0.008; visual mesh filename=package://rethink_ee_description/meshes/electric_gripper/fi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
- link r_gripper_r_finger: geometry collision box size=0.01 0.0135 0.1127; collision box size=0.01 0.05 0.017
- link r_gripper_r_finger_tip: geometry collision cylinder length=0.037 radius=0.008; visual mesh filename=package://rethink_ee_description/meshes/electric_gripper/fi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
- link torso: geometry collision cylinder length=0.7 radius=0.27; visual mesh filename=package://baxter_description/meshes/torso/base_link.DAE
Joints:
- added joint left_gripper_mass: type fixed, parent left_hand, child left_gripper_mass, origin xyz=0.0 0.0 0.0240000000000000 rpy=0.0 0.0 0.0
- added joint left_gripper_object_mass: type fixed, parent left_gripper_mass, child left_gripper_object_mass, origin xyz=0.0 0.0 0.0450000000000000 rpy=0.0 0.0 0.0
- added joint right_gripper_mass: type fixed, parent right_hand, child right_gripper_mass, origin xyz=0.0 0.0 0.0240000000000000 rpy=0.0 0.0 0.0
- added joint right_gripper_object_mass: type fixed, parent right_gripper_mass, child right_gripper_object_mass, origin xyz=0.0 0.0 0.0450000000000000 rpy=0.0 0.0 0.0
- joint left_torso_arm_mount: origin xyz=0.024645 0.219645 0.118588 rpy=0 0 0.7854 -> xyz=0.025447174775 0.219028201403 0.10797895129 rpy=-0.00234473772502 0.000525456482669 0.780499792738
- joint r_gripper_l_finger_joint: origin xyz=0.0 -0.011 0.02 rpy=0 0 0 -> xyz=0.0 -0.0015 0.02 rpy=0 0 0
- joint r_gripper_l_finger_tip_joint: origin xyz=0.0 0.01725 0.075 rpy=0 0 0 -> xyz=0.0 0.01725 0.1127 rpy=0 0 0
- joint r_gripper_r_finger_joint: origin xyz=0.0 0.011 0.02 rpy=0 0 0 -> xyz=0.0 0.0015 0.02 rpy=0 0 0
- joint r_gripper_r_finger_tip_joint: origin xyz=0.0 -0.01725 0.075 rpy=0 0 0 -> xyz=0.0 -0.01725 0.1127 rpy=0 0 0
- joint right_endpoint: origin xyz=0 0 0.095 rpy=0 0 0 -> xyz=0 0 0.1327 rpy=0 0 0
- joint right_torso_arm_mount: origin xyz=0.024645 -0.219645 0.118588 rpy=0 0 -0.7854 -> xyz=0.0247288398034 -0.220050428085 0.108767751469 rpy=0.0029487654568 0.00610368126069 -0.784090817518
